File: PCB_first_try/battery.sch (KiCad schematic (older format))
At the start: 26 parts

Commit message: ok
Parts:
- U?: symbol lib_pro:ADM8660 -> first_try-rescue:ADM8660-lib_pro
Changed lines of the file:
@@
 EESchema Schematic File Version 4
 LIBS:power
-LIBS:device
 LIBS:74xx
-LIBS:audio
-LIBS:interface
 LIBS:first_try-cache
 EELAYER 26 0
@@
 $Descr A4 11693 8268
 encoding utf-8
-Sheet 4 6
+Sheet 4 7
 Title ""
 Date ""
@@
 Connection ~ 2950 4850
 $Comp
-L lib_pro:ADM8660 U?
+L first_try-rescue:ADM8660-lib_pro U?
 U 1 1 5B0BCE64
 P 8450 1500
