File: PCB_first_try/blade.sch (KiCad schematic (older format))
At the start: 6 parts

Commit message: ok
Parts:
- U?: symbol lib_pro:ct124 -> first_try-rescue:ct124-lib_pro
Changed lines of the file:
@@
 EESchema Schematic File Version 4
 LIBS:power
-LIBS:device
 LIBS:74xx
-LIBS:audio
-LIBS:interface
 LIBS:first_try-cache
 EELAYER 26 0
@@
 $EndDescr
 $Comp
-L lib_pro:ct124 U?
+L first_try-rescue:ct124-lib_pro U?
 U 1 1 5B09E6D0
 P 5250 3900
