File: PCB_first_try/line_detection.sch (KiCad schematic (older format))
At the start: 38 parts

Commit message: ok
Parts:
- U? (x2): symbol lib_pro:Linedetector -> first_try-rescue:Linedetector-lib_pro
- U? (x2): symbol lib_pro:UA741 -> first_try-rescue:UA741-lib_pro
Changed lines of the file:
@@
 EESchema Schematic File Version 4
 LIBS:power
-LIBS:device
 LIBS:74xx
-LIBS:audio
-LIBS:interface
 LIBS:first_try-cache
 EELAYER 26 0
@@
 $EndDescr
 $Comp
-L lib_pro:Linedetector U?
+L first_try-rescue:Linedetector-lib_pro U?
 U 1 1 5B0811BD
 P 1250 2550
@@
 $EndComp
 $Comp
-L lib_pro:UA741 U?
+L first_try-rescue:UA741-lib_pro U?
 U 1 1 5B082BC6
 P 8200 2600
@@
 NoConn ~ 7700 2450
 $Comp
-L lib_pro:Linedetector U?
+L first_try-rescue:Linedetector-lib_pro U?
 U 1 1 5B09A819
 P 1200 4950
@@
 $EndComp
 $Comp
-L lib_pro:UA741 U?
+L first_try-rescue:UA741-lib_pro U?
 U 1 1 5B09A882
 P 8150 5000
