File: PCB_first_try/motor_control.sch (KiCad schematic (older format))
At the start: 28 parts

Commit message: ok
Parts:
- IC? (x2): symbol LM18200T:LM18200T -> first_try-rescue:LM18200T-LM18200T
- U?: symbol lib_pro:ct124 -> first_try-rescue:ct124-lib_pro
Changed lines of the file:
@@
 EESchema Schematic File Version 4
 LIBS:power
-LIBS:device
 LIBS:74xx
-LIBS:audio
-LIBS:interface
 LIBS:first_try-cache
 EELAYER 26 0
@@
 $EndDescr
 $Comp
-L LM18200T:LM18200T IC?
+L first_try-rescue:LM18200T-LM18200T IC?
 U 1 1 5AFDD0C4
 P 5800 2200
@@
 currentsense1
 $Comp
-L LM18200T:LM18200T IC?
+L first_try-rescue:LM18200T-LM18200T IC?
 U 1 1 5AFEC512
 P 5850 4950
@@
 Connection ~ 2350 4450
 $Comp
-L lib_pro:ct124 U?
+L first_try-rescue:ct124-lib_pro U?
 U 1 1 5AFD714A
 P 2050 6400
